Commit message: Fix chassis/wheel ground offset, add trail + footprint viz
Wheels and the chassis's ground-contact math were only correct for the
old thin 0.18m-tall chassis; after making the chassis the tall/thick
body, wheel joints and the base_footprint/skid_plate offsets needed to
scale with chassis_z instead of a fixed wheel_radius, or the chassis
sank into the floor and wheels floated near mid-body.

Also adds a trail_publisher node (breadcrumb of where the robot has
actually driven, as a nav_msgs/Path) and RViz displays for it plus
Nav2's published footprint polygons, so both "where it's been" and
"where it's going" are visible for demos.

Co-Authored-By: Claude Sonnet 5 <noreply@anthropic.com>
Claude-Session: https://claude.ai/code/session_01V58Va3tRRZipkHPhPDoSav

File: ros2_ws/src/libbot_description/urdf/base/base.urdf.xacro (robot description, xacro)
@@ -63,8 +63,17 @@
   <!-- base_footprint: ground projection, required by nav2 / robot_localization conventions -->
   <link name="base_footprint"/>
+  <!-- base_link's own box geometry is centered on its origin (extends
+       +/-chassis_z/2), so lifting that origin to chassis_z/2 above the
+       footprint puts the box's BOTTOM flush with the ground, not
+       wheel_radius, which was only correct back when chassis_z (0.18m)
+       happened to be roughly comparable to wheel_radius. With the
+       0.75m-tall chassis, leaving this at wheel_radius buried ~0.3m of
+       the box below the floor and left the wheels (mounted at base_link's
+       own vertical center, see mecanum_wheel below) floating around
+       mid-body instead of at the bottom. -->
   <joint name="base_footprint_joint" type="fixed">
     <parent link="base_footprint"/>
     <child link="base_link"/>
-    <origin xyz="0 0 ${wheel_radius}" rpy="0 0 0"/>
+    <origin xyz="0 0 ${chassis_z/2}" rpy="0 0 0"/>
   </joint>
   <link name="base_link">
@@ -221,8 +230,11 @@
       <parent link="base_link"/>
       <child link="${prefix}_wheel_link"/>
-      <!-- base_link is already wheel_radius above base_footprint/ground
-           (see base_footprint_joint), so wheel joints need zero additional
-           Z offset for the wheel centers to sit at ground + wheel_radius. -->
-      <origin xyz="${x_off} ${y_off} 0" rpy="0 0 0"/>
+      <!-- base_link's origin is chassis_z/2 above the ground (box bottom
+           flush with the floor, see base_footprint_joint), so wheel
+           centers need to sit wheel_radius above the ground, which is
+           chassis_z/2 below base_link's own origin, not 0. Mounting
+           them at 0 (base_link's vertical center) put them floating
+           around mid-body once the chassis got tall. -->
+      <origin xyz="${x_off} ${y_off} ${wheel_radius - chassis_z/2}" rpy="0 0 0"/>
       <axis xyz="0 1 0"/>
       <!-- effort/velocity limits are required even on a continuous joint:
@@ -261,8 +273,13 @@
     </inertial>
   </link>
+  <!-- Just above base_link's own bottom face (-chassis_z/2), which is
+       flush with the ground, same reasoning as base_footprint_joint
+       and the wheel joints above: offsets here are relative to
+       base_link's origin, not the ground, so this has to track
+       chassis_z too, not a fixed wheel_radius-based offset. -->
   <joint name="skid_plate_joint" type="fixed">
     <parent link="base_link"/>
     <child link="skid_plate_link"/>
-    <origin xyz="0 0 ${-wheel_radius + 0.005}" rpy="0 0 0"/>
+    <origin xyz="0 0 ${-chassis_z/2 + 0.005}" rpy="0 0 0"/>
   </joint>
   <gazebo reference="skid_plate_link">

Commit message: Fix persistent tip-over, flip default spawn orientation 180deg
The earlier inertia-only tip-over fix wasn't enough once the chassis
got tall/heavy from the visual restyle -- confirmed still tipping on
collision during testing. Fixes the actual physics this time: more
realistic mass (35kg, up from 20kg), a low center of gravity (inertial
origin moved down to the bottom quarter of the body, like where a real
AMR's batteries would sit), further-boosted roll/pitch inertia, and a
wider ground-contact skid plate. Verified by ramming the robot into an
obstacle at 0.6 m/s for 8s straight with roll/pitch staying under
0.0002 rad throughout.

Also flips the default spawn yaw 180 degrees per user request.

Co-Authored-By: Claude Sonnet 5 <noreply@anthropic.com>
Claude-Session: https://claude.ai/code/session_01V58Va3tRRZipkHPhPDoSav

File: ros2_ws/src/libbot_description/urdf/base/base.urdf.xacro (robot description, xacro)
@@ -20,5 +20,11 @@
        mast. -->
   <xacro:property name="chassis_z" value="0.75"/>
-  <xacro:property name="chassis_mass" value="20.0"/>
+  <!-- Real AMRs this size run 30-45kg (batteries, motors, compute), and
+       that mass matters here: it's not just "heavier feels more real",
+       more mass directly means more rotational inertia (I scales with
+       mass), which is what actually resists a collision's angular
+       impulse and keeps the robot from tipping. See base_link's
+       <inertial> below for the other half of the fix (a low CoG). -->
+  <xacro:property name="chassis_mass" value="35.0"/>
   <xacro:property name="wheel_radius" value="0.075"/>
   <xacro:property name="wheel_width" value="0.05"/>
@@ -92,20 +98,27 @@
     </collision>
     <inertial>
-      <origin xyz="0 0 0" rpy="0 0 0"/>
+      <!-- Real service robots put batteries/heavy components low in the
+           chassis specifically to keep the center of gravity low and
+           resist tipping. This is the actual physical fix, not just a
+           bigger-number hack. Offsetting the inertial origin down to
+           near the bottom quarter of the 0.75m-tall box (rather than
+           the box's geometric center at z=0) simulates that: the
+           restoring gravity torque when something pushes the top of the
+           robot scales with how far the CoG has to swing sideways
+           before it crosses the support base's edge, and a lower CoG
+           makes that swing much larger for the same tip angle. -->
+      <origin xyz="0 0 -0.25" rpy="0 0 0"/>
       <mass value="${chassis_mass}"/>
-      <!-- Roll/pitch (ixx/iyy) are boosted well above the box's natural
-           values (~0.22/0.33) instead of using box_inertia directly. The
-           ~0.85m mast puts the lidar/camera roughly a meter above the
-           chassis; a collision up there (driving into a desk, teleop
-           misjudging clearance) applies its force at that height, and
-           against the base's actual (fairly narrow, ~0.4-0.5m) footprint
-           that's enough torque to physically tip a normal-inertia chassis
-           over, which happened during mapping testing. Yaw (izz) is left
-           at its natural value so turning stays responsive; only the
-           tip-over axes are stiffened, standing in for what a real base
-           would get from a low, wide chassis or active gyro stabilization
-           without redesigning the footprint the user asked to keep narrow
-           enough for the aisles. -->
-      <inertia ixx="2.5" ixy="0.0" ixz="0.0" iyy="3.5" iyz="0.0" izz="0.4783"/>
+      <!-- Roll/pitch (ixx/iyy) are additionally boosted above the box's
+           natural values instead of using box_inertia directly. The
+           sensor puck/camera sit roughly a meter up, and a collision
+           there (driving into a desk, teleop misjudging clearance)
+           applies force at that height. A first pass at this (lower
+           mass, CoG at box center) still tipped over during testing;
+           this combines the low CoG above with higher inertia and more
+           realistic mass for AMRs this size. Yaw (izz) is left at its
+           natural value so turning stays responsive; only the tip-over
+           axes are stiffened. -->
+      <inertia ixx="6.0" ixy="0.0" ixz="0.0" iyy="8.0" iyz="0.0" izz="1.196"/>
     </inertial>
   </link>
@@ -264,7 +277,12 @@
        simple, uniform-friction contact patch removes that interference
        entirely. See README "Drivetrain design note" for the full story. -->
+  <!-- Widened from 0.85x to 0.95x chassis footprint. A wider ground
+       contact patch means the robot has to rotate further before its
+       (now much lower, see base_link inertial) CoG swings past the
+       support edge, adding margin against tipping on top of the mass/
+       inertia changes above. -->
   <link name="skid_plate_link">
     <collision>
-      <geometry><box size="${chassis_x*0.85} ${chassis_y*0.85} 0.01"/></geometry>
+      <geometry><box size="${chassis_x*0.95} ${chassis_y*0.95} 0.01"/></geometry>
     </collision>
     <inertial>
