Commit message: Fix item markers to derive map position live, add basket walls
Root cause of markers showing "totally wrong" positions: an earlier
fix anchored a `world` frame to `odom` via a *hardcoded* spawn-pose
offset (simulation.launch.py's x/y/yaw), assuming odom's origin never
moves from that spawn pose. That's false the moment anything teleports
the robot without also resetting the odometry plugin's internal
integrator (e.g. the control panel's "Reset Position" button) --
confirmed live: odom->base_footprint was reporting the *spawn*
coordinates instead of ~0, meaning the hardcoded assumption had gone
stale.

Rewrote item_pose_publisher to compute map -> item fresh every cycle
from two live facts instead, no fixed assumptions:
  - this robot's own ground-truth pose in Gazebo's world frame (same
    /libbot/model_states message, filtering for robot_model_name)
  - a live TF lookup of map -> base_footprint (the exact same
    transform Nav2 itself resolves through)
map_to_item = map_to_base @ inverse(world_to_base) @ world_to_item

This also directly satisfies "same transform as nav2" -- both draw
from the identical map->base_footprint source, so a task manager can
send NavigateToPose goals straight at these item positions. Verified
live: book position closely tracks raw ground truth with sub-cm
jitter, self-consistent with the robot's own resolved map position.

Also: book_tray_link (the basket) now has actual walls (floor + 4
thin sides) instead of being a bare flat plate, same 0.16x0.24
footprint as before so the robot's overall size/silhouette is
unchanged. Removed simulation.launch.py's now-unused spawn_x/y/yaw
params passed to item_pose_publisher.

Co-Authored-By: Claude Sonnet 5 <noreply@anthropic.com>
Claude-Session: https://claude.ai/code/session_01UEWnJt5f5knTzkV3i2xv6u

File: ros2_ws/src/libbot_description/urdf/base/payload_platform.urdf.xacro (robot description, xacro)
@@ -31,6 +31,12 @@
     <origin xyz="0 0 ${chassis_z/2 + mast_height/2}" rpy="0 0 0"/>
   </joint>
-  <!-- Book intake tray on the front, at an accessible low-middle height
-       on the body rather than tracking the (now much taller) body top. -->
+  <!-- Book collection basket on the front, at an accessible low-middle
+       height on the body. Same 0.16 x 0.24 footprint as the flat tray
+       this replaces (no change to the robot's overall size/silhouette),
+       just floor + 4 thin walls on that same footprint so books
+       book_sorter_node.py attaches here visually sit inside a basket
+       instead of floating on a bare plate. -->
+  <xacro:property name="basket_wall_h" value="0.08"/>
+  <xacro:property name="basket_wall_t" value="0.01"/>
   <link name="book_tray_link">
     <visual>
@@ -40,4 +46,42 @@
     <collision>
       <geometry><box size="0.16 0.24 0.02"/></geometry>
+    </collision>
+    <!-- Front/back walls (span y, thin in x) -->
+    <visual>
+      <origin xyz="0.075 0 ${0.01 + basket_wall_h/2}" rpy="0 0 0"/>
+      <geometry><box size="${basket_wall_t} 0.24 ${basket_wall_h}"/></geometry>
+      <material name="libbot_body_teal"/>
+    </visual>
+    <collision>
+      <origin xyz="0.075 0 ${0.01 + basket_wall_h/2}" rpy="0 0 0"/>
+      <geometry><box size="${basket_wall_t} 0.24 ${basket_wall_h}"/></geometry>
+    </collision>
+    <visual>
+      <origin xyz="-0.075 0 ${0.01 + basket_wall_h/2}" rpy="0 0 0"/>
+      <geometry><box size="${basket_wall_t} 0.24 ${basket_wall_h}"/></geometry>
+      <material name="libbot_body_teal"/>
+    </visual>
+    <collision>
+      <origin xyz="-0.075 0 ${0.01 + basket_wall_h/2}" rpy="0 0 0"/>
+      <geometry><box size="${basket_wall_t} 0.24 ${basket_wall_h}"/></geometry>
+    </collision>
+    <!-- Left/right walls (span x, thin in y) -->
+    <visual>
+      <origin xyz="0 0.115 ${0.01 + basket_wall_h/2}" rpy="0 0 0"/>
+      <geometry><box size="0.16 ${basket_wall_t} ${basket_wall_h}"/></geometry>
+      <material name="libbot_body_teal"/>
+    </visual>
+    <collision>
+      <origin xyz="0 0.115 ${0.01 + basket_wall_h/2}" rpy="0 0 0"/>
+      <geometry><box size="0.16 ${basket_wall_t} ${basket_wall_h}"/></geometry>
+    </collision>
+    <visual>
+      <origin xyz="0 -0.115 ${0.01 + basket_wall_h/2}" rpy="0 0 0"/>
+      <geometry><box size="0.16 ${basket_wall_t} ${basket_wall_h}"/></geometry>
+      <material name="libbot_body_teal"/>
+    </visual>
+    <collision>
+      <origin xyz="0 -0.115 ${0.01 + basket_wall_h/2}" rpy="0 0 0"/>
+      <geometry><box size="0.16 ${basket_wall_t} ${basket_wall_h}"/></geometry>
     </collision>
     <inertial>

Commit message: Fix basket mounted inside the chassis instead of protruding from it
book_tray_joint's x (0.14) was well inside the chassis's own front
face (chassis_x/2=0.25, chassis_x=0.50) and z (-0.125) was well
within its vertical extent (spans -0.375 to +0.375) -- the basket was
entirely embedded in the solid chassis box the whole time, invisible
from outside and, worse, the same teal material as the chassis
itself, so it just read as "one big box" with the basket hidden
inside it. Moved x to chassis_x/2 + half the basket's own depth so it
actually protrudes from the front face instead.

Also: full clean rebuild (rm -rf build install log + colcon build)
per request, and committing the newly saved half_map.

Co-Authored-By: Claude Sonnet 5 <noreply@anthropic.com>
Claude-Session: https://claude.ai/code/session_01UEWnJt5f5knTzkV3i2xv6u

File: ros2_ws/src/libbot_description/urdf/base/payload_platform.urdf.xacro (robot description, xacro)
@@ -93,5 +93,12 @@
     <parent link="base_link"/>
     <child link="book_tray_link"/>
-    <origin xyz="0.14 0 ${-chassis_z/2 + 0.25}" rpy="0 0 0"/>
+    <!-- x was 0.14, well inside the chassis's own front face at
+         chassis_x/2=0.25 (chassis_x=0.50): the basket was entirely
+         embedded in the solid chassis box, invisible from outside
+         (same teal material as the chassis besides). Mounted just
+         proud of the front face instead so it actually protrudes and
+         is visible: chassis_x/2 + half the basket's own depth
+         (0.16/2=0.08), i.e. flush against the face. -->
+    <origin xyz="${chassis_x/2 + 0.08} 0 ${-chassis_z/2 + 0.25}" rpy="0 0 0"/>
   </joint>
   <gazebo reference="sensor_mast_link">
