Commit message: Fix arm gripper_link lumping and stabilize book pick/place in Gazebo sim
gripper_link was silently getting fused into wrist_link by URDF->SDF
conversion despite disableFixedJointLumping (unsupported by this
sdformat build); switched to a zero-range revolute joint, which is never
lumped, so gripper_link exists as a real link the attacher plugin can
grab.

The attach/detach plugin itself had three compounding bugs verified live
in Gazebo: missing the physics-engine update mutex around joint
mutation (wedged the whole world on a second attach/detach call), leaf
link names not matching AWS RoboMaker props' flattened <include> naming
(gripper_link/book link never found), and a dynamically created ODE
fixed joint between two independent top-level models resonating into a
runaway tumble within a couple of physics steps regardless of mass/pose
fixups. Replaced the joint with a plain per-step kinematic pose-follow
(book stays static, teleported to track the gripper each world update),
which sidesteps the constraint solver entirely. Verified end-to-end in a
live headless sim: attach, multi-waypoint arm carry, detach (book rests
exactly in place), and repeated attach/detach all succeed with no
explosions or hangs.

File: ros2_ws/src/libbot_description/urdf/arm/arm.urdf.xacro (robot description, xacro)
@@ -153,17 +153,21 @@
     </inertial>
   </link>
-  <joint name="gripper_joint" type="fixed">
+  <!-- Zero-range revolute rather than type="fixed": Gazebo Classic's
+       URDF->SDF conversion lumps any fixed-jointed child link's geometry
+       into its parent (gripper_link would stop existing as its own SDF
+       link), and <disableFixedJointLumping> does not suppress this on the
+       sdformat version this project builds against. A revolute joint is
+       never lumped regardless, and clamping its range to [0, 0] makes it
+       behave exactly like a fixed joint. libbot_gazebo_plugins' attach/
+       detach services need gripper_link addressable as a real link to
+       weld a book to it. -->
+  <joint name="gripper_joint" type="revolute">
     <parent link="wrist_link"/>
     <child link="gripper_link"/>
     <origin xyz="0.09 0 0" rpy="0 0 0"/>
+    <axis xyz="0 0 1"/>
+    <limit lower="0" upper="0" effort="0" velocity="0"/>
+    <dynamics damping="0.0" friction="0.0"/>
   </joint>
-  <!-- Without this, Gazebo Classic's URDF->SDF conversion lumps
-       gripper_link's geometry into wrist_link (standard behavior for any
-       fixed joint) and gripper_link stops existing as its own SDF link.
-       libbot_gazebo_plugins' attach/detach services need gripper_link to
-       be addressable as a real link to weld a book to it. -->
-  <gazebo reference="gripper_link">
-    <disableFixedJointLumping>true</disableFixedJointLumping>
-  </gazebo>
   <gazebo reference="arm_base_link"><material>Gazebo/Grey</material></gazebo>
   <gazebo reference="shoulder_pan_link"><material>Gazebo/Grey</material></gazebo>

Commit message: Fix Nav2 movement/localization, side-mount the arm, add FAST-LIO2 3D localization
Nav2 was silently unable to move the robot at all: behavior_server's
Spin/BackUp/DriveOnHeading recoveries publish plain Twist on the default
/cmd_vel, which nothing subscribes to -- only controller_server had the
remap onto the mecanum controller's actual command topic. Added the same
remap to behavior_server.

AMCL's initial_pose.yaw (1.5708) was stale against the robot's actual
spawn yaw (-1.5708, flipped 180deg in an earlier commit but never
mirrored into amcl.yaml), seeding the particle filter facing the wrong
way on every run -- the likely cause of "map doesn't align with live
data" in a mostly-symmetric library layout.

task_manager_node.py was missing its executable bit, so
`collect_books:=true` failed outright with "executable not found".

Arm remounted from the front-top edge (where it visually collided with
the chassis fascia) to the chassis's -Y side face.

Added FAST-LIO2 (LiDAR-IMU odometry) as a real 3D localization demo
using the robot's existing 3D lidar + IMU, chosen over a full SLAM stack
(rtabmap) specifically for being light enough to target a Jetson Nano
Super eventually. Needed two adaptations for the simulated sensor: a
small adapter node synthesizes the ring/time per-point fields Gazebo's
ray sensor doesn't provide, and the lidar was raised further above the
sensor mast (it was still clipping the mast/fascia in its own downward
FOV). Built from source in a separate ~/fastlio_ws overlay (FAST_LIO's
ROS2 branch + livox_ros_driver2, needed only for message-type headers)
since it isn't packaged for apt; see README "3D localization" for the
build steps.

README updated to match current reality: the old RFID/sorting system
description (removed in an earlier commit) is gone, arm-based pick/place
and 3D localization are documented, and two screenshots show the robot
and FAST-LIO2 tracking a live trajectory.

File: ros2_ws/src/libbot_description/urdf/arm/arm.urdf.xacro (robot description, xacro)
@@ -31,8 +31,15 @@
     </inertial>
   </link>
+  <!-- Side-mounted (on the -Y side, opposite chassis_side_panel_link on
+       +Y in base.urdf.xacro) rather than perched on the front-top edge,
+       where it visually collided with chassis_fascia_link. No yaw
+       rotation: the arm's local +X ("reach" direction, see all the link
+       visual/collision offsets below) still points straight forward,
+       exactly as when it was front-mounted, so the canned joint poses in
+       libbot_manipulation/task_manager_node.py need no changes. -->
   <joint name="arm_base_joint" type="fixed">
     <parent link="base_link"/>
     <child link="arm_base_link"/>
-    <origin xyz="${chassis_x/2 - 0.08} 0 ${chassis_z/2 + 0.03}" rpy="0 0 0"/>
+    <origin xyz="0.05 ${-(chassis_y/2 + 0.03)} ${chassis_z/2 - 0.05}" rpy="0 0 0"/>
   </joint>
   <!-- shoulder_pan: yaw about the arm base -->

File: ros2_ws/src/libbot_description/urdf/libbot.urdf.xacro (robot description, xacro)
@@ -10,5 +10,8 @@
   <xacro:include filename="$(find realsense2_description)/urdf/_d435i.urdf.xacro"/>
   <xacro:libbot_imu parent="base_link" xyz="0 0 ${chassis_z/2 + 0.01}"/>
-  <xacro:libbot_lidar_3d parent="sensor_mast_link" xyz="0 0 ${mast_height/2 + 0.03}" hz="5"/>
+  <!-- Raised well above the sensor-mast puck top (was only 0.03m above
+       it, so the lidar's own downward FOV rays clipped the mast/chassis
+       fascia at short range, especially once the robot started moving). -->
+  <xacro:libbot_lidar_3d parent="sensor_mast_link" xyz="0 0 ${mast_height/2 + 0.15}" hz="5"/>
   <!-- RealSense D435i mounted forward-facing on the chassis's upper
        front face at roughly mid-shelf height, angled down slightly to
