Commit message: Add manipulation stack: arm URDF, Gazebo link-attacher plugin, task manager
Introduces libbot_manipulation (task manager node, book/shelf catalogs)
and libbot_gazebo_plugins (link attacher service) to support picking and
placing books, plus the supporting arm URDF, controller, and world updates.

File: ros2_ws/src/libbot_description/urdf/control/ros2_control.urdf.xacro (robot description, xacro)
@@ -6,4 +6,14 @@
         <param name="min">-30</param>
         <param name="max">30</param>
+      </command_interface>
+      <state_interface name="position"/>
+      <state_interface name="velocity"/>
+    </joint>
+  </xacro:macro>
+  <xacro:macro name="libbot_arm_ros2_control_joint" params="name lower upper">
+    <joint name="${name}">
+      <command_interface name="position">
+        <param name="min">${lower}</param>
+        <param name="max">${upper}</param>
       </command_interface>
       <state_interface name="position"/>
@@ -19,4 +29,8 @@
     <xacro:libbot_wheel_ros2_control_joint name="rear_left"/>
     <xacro:libbot_wheel_ros2_control_joint name="rear_right"/>
+    <xacro:libbot_arm_ros2_control_joint name="shoulder_pan_joint" lower="-2.0" upper="2.0"/>
+    <xacro:libbot_arm_ros2_control_joint name="shoulder_lift_joint" lower="-1.6" upper="1.2"/>
+    <xacro:libbot_arm_ros2_control_joint name="elbow_joint" lower="-2.2" upper="1.8"/>
+    <xacro:libbot_arm_ros2_control_joint name="wrist_pitch_joint" lower="-1.6" upper="1.6"/>
   </ros2_control>
   <gazebo>

File: ros2_ws/src/libbot_description/urdf/libbot.urdf.xacro (robot description, xacro)
@@ -4,4 +4,5 @@
   <xacro:include filename="$(find libbot_description)/urdf/base/base.urdf.xacro"/>
   <xacro:include filename="$(find libbot_description)/urdf/base/payload_platform.urdf.xacro"/>
+  <xacro:include filename="$(find libbot_description)/urdf/arm/arm.urdf.xacro"/>
   <xacro:include filename="$(find libbot_description)/urdf/sensors/imu.urdf.xacro"/>
   <xacro:include filename="$(find libbot_description)/urdf/sensors/lidar_3d.urdf.xacro"/>

Commit message: Replace AMCL with FAST-LIO2 as Nav2's localization source; fix arm TF gap
Running AMCL and FAST-LIO2 simultaneously was redundant (both estimate
global pose). FAST-LIO2 now provides Nav2's map->odom transform directly:
fastlio_map_odom_bridge.py composes FAST-LIO2's pose estimate with the
EKF's existing odom->base_footprint (map->odom = map->body *
inverse(odom->base_footprint)), preserving local costmap continuity the
same way AMCL's correction did. localization_fastlio.launch.py bundles
map_server (costmaps still need the static map) + the 3D lidar adapter +
FAST-LIO2 + the bridge; localization.launch.py's use_amcl flag (kept for
backward compatibility with existing callers) now routes to this instead
of bare AMCL. nav2_amcl dependency and amcl.yaml removed.

Also fixes a real bug this surfaced: gripper_joint (made a zero-range
revolute joint in an earlier commit, to stop Gazebo's URDF->SDF lumping)
was never registered in ros2_control, so joint_state_broadcaster never
reported its state and robot_state_publisher silently dropped
wrist_link->gripper_link from TF entirely -- breaking RobotModel
rendering for the arm past the wrist and anything the link-attacher
plugin welds there. Registered as a state-only (no command_interface)
joint so it's included in joint_state_broadcaster's output like every
other joint.

File: ros2_ws/src/libbot_description/urdf/control/ros2_control.urdf.xacro (robot description, xacro)
@@ -21,4 +21,17 @@
     </joint>
   </xacro:macro>
+  <!-- State-only (no command_interface): gripper_joint is a zero-range
+       revolute joint (arm.urdf.xacro), never actively driven, but it
+       still needs to be registered here so joint_state_broadcaster
+       reports it, since otherwise robot_state_publisher never receives
+       a state for it and silently drops wrist_link to gripper_link from
+       TF entirely, breaking RobotModel rendering for the whole arm past
+       the wrist (and anything the link-attacher plugin welds there). -->
+  <xacro:macro name="libbot_passive_ros2_control_joint" params="name">
+    <joint name="${name}">
+      <state_interface name="position"/>
+      <state_interface name="velocity"/>
+    </joint>
+  </xacro:macro>
   <ros2_control name="libbot_gazebo_system" type="system">
     <hardware>
@@ -33,4 +46,5 @@
     <xacro:libbot_arm_ros2_control_joint name="elbow_joint" lower="-2.2" upper="1.8"/>
     <xacro:libbot_arm_ros2_control_joint name="wrist_pitch_joint" lower="-1.6" upper="1.6"/>
+    <xacro:libbot_passive_ros2_control_joint name="gripper_joint"/>
   </ros2_control>
   <gazebo>
