Commit message: Smooth ICP jitter, add shelf markers, fix lidar mount, add book sorting
- fastlio_map_odom_bridge: exponential smoothing + outlier rejection on
  the ICP-derived map->odom correction. It was applying each new
  registration's x/y/yaw raw with no filtering, which visibly jittered
  everything under `map` (including the new item markers) and let a
  single bad registration snap the whole map frame to a wrong pose.

- item_pose_publisher: also tracks BookshelfA_01_001..004 (the center
  shelves) as larger blue cube markers, distinct from the small orange
  book markers, using the same live TF/marker mechanism.

- libbot.urdf.xacro: the 3D lidar is now shifted 0.04m forward, and a
  new cosmetic standoff link (lidar_riser_link) fills the gap between
  the sensor-mast puck and the lidar mount point, fixing the "floating"
  look. The lidar's actual mount height is unchanged (it's deliberately
  above the puck to avoid its downward FOV clipping the puck, per the
  existing comment there) -- only the visual connection and x position
  changed, no existing link was resized.

- New book_sorter_node.py (libbot_manipulation): same pick/place
  mechanics as task_manager_node.py, but scoped to specific book_names
  (default the four currently-tracked books) and shelf_names (the four
  center shelves), and attaches picked books to book_tray_link -- the
  existing front intake tray, reused as-is with no geometry changes --
  instead of directly to gripper_link, so it reads as "collected into a
  basket" between pickup and drop-off. Both name lists are runtime-
  settable parameters, matching item_pose_publisher's convention, so
  more books can be added later without a restart.

- New "Sort Books" button in the RViz control panel triggers it
  (requires Navigation already running).

Co-Authored-By: Claude Sonnet 5 <noreply@anthropic.com>
Claude-Session: https://claude.ai/code/session_01UEWnJt5f5knTzkV3i2xv6u

File: ros2_ws/src/libbot_description/urdf/libbot.urdf.xacro (robot description, xacro)
@@ -10,8 +10,35 @@
   <xacro:include filename="$(find realsense2_description)/urdf/_d435i.urdf.xacro"/>
   <xacro:libbot_imu parent="base_link" xyz="0 0 ${chassis_z/2 + 0.01}"/>
+  <!-- Riser between the mast puck top and the lidar: purely cosmetic
+       (thin standoff cylinder, no functional role), added because the
+       lidar's mount height is deliberately well above the puck (next
+       block down), which otherwise reads as the lidar floating
+       disconnected above the robot rather than mounted on it. -->
+  <link name="lidar_riser_link">
+    <visual>
+      <geometry><cylinder radius="0.05" length="0.12"/></geometry>
+      <material name="libbot_wheel_black"/>
+    </visual>
+    <inertial>
+      <mass value="0.05"/>
+      <inertia ixx="1e-5" ixy="0" ixz="0" iyy="1e-5" iyz="0" izz="1e-5"/>
+    </inertial>
+  </link>
+  <joint name="lidar_riser_joint" type="fixed">
+    <parent link="sensor_mast_link"/>
+    <child link="lidar_riser_link"/>
+    <!-- Spans mast top (z=mast_height/2=0.06) up to the lidar's bottom
+         face (lidar origin 0.21 minus its own half-height 0.03 = 0.18),
+         so length=0.12 centered at z=0.12 (=mast_height/2+0.06) touches
+         both with no gap, under the lidar's own forward-shifted x value. -->
+    <origin xyz="0.04 0 ${mast_height/2 + 0.06}" rpy="0 0 0"/>
+  </joint>
   <!-- Raised well above the sensor-mast puck top (was only 0.03m above
        it, so the lidar's own downward FOV rays clipped the mast/chassis
-       fascia at short range, especially once the robot started moving). -->
-  <xacro:libbot_lidar_3d parent="sensor_mast_link" xyz="0 0 ${mast_height/2 + 0.15}" hz="5"/>
+       fascia at short range, especially once the robot started moving);
+       kept unchanged, only x shifted slightly forward per request, with
+       the riser above now visually connecting it to the puck instead of
+       leaving a bare gap. -->
+  <xacro:libbot_lidar_3d parent="sensor_mast_link" xyz="0.04 0 ${mast_height/2 + 0.15}" hz="5"/>
   <!-- RealSense D435i mounted forward-facing on the chassis's upper
        front face at roughly mid-shelf height, angled down slightly to
